Commit message: double ackermann controller for rover

File: install/rover_description/share/rover_description/urdf/kratos_rover.urdf.xacro (robot description, xacro)
@@ -1,86 +1,24 @@
 <?xml version="1.0"?>
 <robot xmlns:xacro="http://www.ros.org/wiki/xacro" name="kratos_rover">
-    <xacro:include filename="inertial_macros.xacro"/>
     <xacro:property name="chassis_len" value="0.5"/>
     <xacro:property name="chassis_width" value="0.3"/>
     <xacro:property name="chassis_height" value="0.1"/>
-    <xacro:property name="wheel_radius" value="0.10"/>
+    <xacro:property name="wheel_radius" value="0.12"/>
     <xacro:property name="wheel_width" value="0.08"/>
-    <xacro:property name="wheel_x_offset" value="0.2"/>  <xacro:property name="wheel_y_offset" value="0.25"/> <xacro:property name="steer_z_offset" value="-0.05"/> <xacro:property name="steer_limit" value="1.57"/>
+    <xacro:property name="wheel_x_offset" value="0.2"/>
+    <xacro:property name="wheel_y_offset" value="0.3"/>
+    <xacro:property name="steer_z_offset" value="-0.05"/>
+    <xacro:property name="steer_limit" value="3.14"/>
     <material name="gray"><color rgba="0.6 0.6 0.6 1.0"/></material>
     <material name="black"><color rgba="0.1 0.1 0.1 1.0"/></material>
     <material name="blue"><color rgba="0.0 0.3 0.8 1.0"/></material>
-    <link name="base_footprint"/>
-    <joint name="base_joint" type="fixed">
-        <parent link="base_footprint"/>
-        <child link="base_link"/>
-        <origin xyz="0 0 0.21" rpy="0 0 0"/>
-    </joint>
-    <link name="base_link">
-        <visual>
-            <origin xyz="0 0 0" rpy="0 0 0"/>
-            <geometry>
-                <box size="${chassis_len} ${chassis_width} ${chassis_height}"/>
-            </geometry>
-            <material name="gray"/>
-        </visual>
-        <collision>
-            <origin xyz="0 0 0" rpy="0 0 0"/>
-            <geometry>
-                <box size="${chassis_len} ${chassis_width} ${chassis_height}"/>
-            </geometry>
-        </collision>
-        <xacro:inertial_box mass="15.0" x="${chassis_len}" y="${chassis_width}" z="${chassis_height}">
-            <origin xyz="0 0 0" rpy="0 0 0"/>
-        </xacro:inertial_box>
-    </link>
-    <xacro:macro name="swerve_wheel" params="prefix x_reflect y_reflect">
-        <link name="${prefix}_steer_link">
-            <visual>
-                <origin xyz="0 0 0" rpy="0 0 0"/>
-                <geometry>
-                    <cylinder radius="0.02" length="0.04"/>
-                </geometry>
-                <material name="blue"/>
-            </visual>
-            <xacro:inertial_cylinder mass="0.5" length="0.04" radius="0.02">
-                <origin xyz="0 0 0" rpy="0 0 0"/>
-            </xacro:inertial_cylinder>
-        </link>
-        <joint name="${prefix}_steer_joint" type="revolute">
-            <parent link="base_link"/>
-            <child link="${prefix}_steer_link"/>
-            <origin xyz="${x_reflect * wheel_x_offset} ${y_reflect * wheel_y_offset} ${steer_z_offset}" rpy="0 0 0"/>
-            <axis xyz="0 0 1"/>
-            <limit lower="-${steer_limit}" upper="${steer_limit}" effort="10.0" velocity="2.0"/>
-        </joint>
-        <link name="${prefix}_wheel_link">
-            <visual>
-                <origin xyz="0 0 0" rpy="${pi/2} 0 0"/>
-                <geometry>
-                    <cylinder radius="${wheel_radius}" length="${wheel_width}"/>
-                </geometry>
-                <material name="black"/>
-            </visual>
-            <collision>
-                <origin xyz="0 0 0" rpy="${pi/2} 0 0"/>
-                <geometry>
-                    <cylinder radius="${wheel_radius}" length="${wheel_width}"/>
-                </geometry>
-            </collision>
-            <xacro:inertial_cylinder mass="1.5" length="${wheel_width}" radius="${wheel_radius}">
-                <origin xyz="0 0 0" rpy="${pi/2} 0 0"/>
-            </xacro:inertial_cylinder>
-        </link>
-        <joint name="${prefix}_drive_joint" type="continuous">
-            <parent link="${prefix}_steer_link"/>
-            <child link="${prefix}_wheel_link"/>
-            <origin xyz="0 0 -0.04" rpy="0 0 0"/>
-            <axis xyz="0 1 0"/>
-        </joint>
-    </xacro:macro>
+    <xacro:include filename="inertial_macros.xacro"/>
+    <xacro:include filename="core_chassis.xacro"/>
+    <xacro:include filename="wheel_macro.xacro"/>
     <xacro:swerve_wheel prefix="fl" x_reflect="1" y_reflect="1"/>
     <xacro:swerve_wheel prefix="fr" x_reflect="1" y_reflect="-1"/>
     <xacro:swerve_wheel prefix="rl" x_reflect="-1" y_reflect="1"/>
     <xacro:swerve_wheel prefix="rr" x_reflect="-1" y_reflect="-1"/>
+    <xacro:include filename="ros2_control.xacro"/>
+    <xacro:include filename="gazebo_plugins.xacro"/>
 </robot>
