Commit message: added gitignore

File: src/rover_description/urdf/kratos_rover.urdf.xacro (robot description, xacro)
@@ -9,5 +9,5 @@
     <xacro:property name="wheel_y_offset" value="0.3"/>
     <xacro:property name="steer_z_offset" value="-0.05"/>
-    <xacro:property name="steer_limit" value="3.14"/>
+    <xacro:property name="steer_limit" value="1.57"/>
     <material name="gray"><color rgba="0.6 0.6 0.6 1.0"/></material>
     <material name="black"><color rgba="0.1 0.1 0.1 1.0"/></material>

File: src/rover_description/urdf/ros2_control.xacro (robot description, xacro)
@@ -8,6 +8,6 @@
             <joint name="${prefix}_steer_joint">
                 <command_interface name="position"/>
-                    <param name="min">-90</param>
-                    <param name="max">90</param>
+                    <param name="min">-1.5708</param>
+                    <param name="max">1.5708</param>
                 <state_interface name="position"/>
             </joint>
